Commit message: added lidar transforms

File: urdf/a2.urdf (robot description, URDF)
Before this commit: robot a2, 19 links, 18 joints
Joints:
- joint lidar_joint: origin xyz=0.0 0.0 0.2 rpy=0 0 0 -> xyz=0.33767 0.0 0.08134 rpy=1.5708 0.0 1.5708

Commit message: Removing inertia of base_link to avoid error
@TODO: This needs to be fixed differently, as mass and inertia are need in sim

File: urdf/a2.urdf (robot description, URDF)
Before this commit: robot a2, 19 links, 18 joints
Links:
- link base_link: mass 19.651 -> None

Commit message: added rear lidar

File: urdf/a2.urdf (robot description, URDF)
Before this commit: robot a2, 19 links, 18 joints
Links:
- removed link lidar_link
- added link front_lidar_link, mass 0.001
- added link rear_lidar_link, mass 0.001
Joints:
- removed joint lidar_joint
- added joint front_lidar_joint: type fixed, parent base_link, child front_lidar_link, origin xyz=0.33767 0.0 0.08134 rpy=1.5708 0.0 1.5708
- added joint rear_lidar_joint: type fixed, parent base_link, child rear_lidar_link, origin xyz=-0.27997 0.0 0.087337 rpy=1.5708 0.0 -1.5708

Commit message: updated camera link position

File: urdf/a2.urdf (robot description, URDF)
Before this commit: robot a2, 20 links, 19 joints
Links:
- added link camera_link, mass 0.001
Joints:
- added joint front_camera_joint: type fixed, parent base_link, child camera_link, origin xyz=0.3421785 0.0336742 0.0513862 rpy=1.5708 0.0 1.5708

Commit message: Revert "fixed camera joint"
This reverts commit 958101c1d1b3220b1a642196bdd7d47d384424ef.

File: urdf/a2.urdf (robot description, URDF)
Before this commit: robot a2, 22 links, 21 joints
Links:
- removed link front_camera_optical_frame
Joints:
- removed joint front_camera_optical_joint
- joint front_camera_joint: origin xyz=0.3421785 0.0336742 0.0513862 rpy=0.0 0.0 0.0 -> xyz=0.3421785 0.0336742 0.0513862 rpy=1.5708 0.0 1.5708

Commit message: Revert "updated camera link position"
This reverts commit cecde194e45cdd98cfaecbe109f9891cc72b6e80.

File: urdf/a2.urdf (robot description, URDF)
Before this commit: robot a2, 21 links, 20 joints
Links:
- removed link camera_link
Joints:
- removed joint front_camera_joint

Commit message: dlio works in sim

File: urdf/a2.urdf (robot description, URDF)
Before this commit: robot a2, 22 links, 21 joints
Links:
- added link front_lidar_imu_link, mass 0.001
Joints:
- added joint front_lidar_imu_joint: type fixed, parent base_link, child front_lidar_imu_link, origin xyz=0.34629 -0.00914 0.04218 rpy=1.5708 0.0 1.5708

Commit message: convert STL to stl format (fix for mac)

File: urdf/a2.urdf (robot description, URDF)
Before this commit: robot a2, 23 links, 22 joints
Links:
- link FL_calf: geometry collision box size=0.01 0.036 0.06; collision box size=0.02 0.036 0.06
- link FL_foot: geometry collision sphere radius=0.032; visual mesh filename=package://a2_description/meshes/left_front_Link4.stl
- link FL_hip: geometry visual mesh filename=package://a2_description/meshes/left_front_Link1.stl
- link FL_thigh: geometry collision box size=0.017 0.05 0.05; collision box size=0.055 0.036 0.17
- link FR_calf: geometry collision box size=0.01 0.036 0.06; collision box size=0.02 0.036 0.06
- link FR_foot: geometry collision sphere radius=0.032; visual mesh filename=package://a2_description/meshes/right_front_Link4.stl
- link FR_hip: geometry visual mesh filename=package://a2_description/meshes/right_front_Link1.stl
- link FR_thigh: geometry collision box size=0.017 0.05 0.05; collision box size=0.055 0.036 0.17
- link RL_calf: geometry collision box size=0.01 0.036 0.06; collision box size=0.02 0.036 0.06
- link RL_foot: geometry collision sphere radius=0.032; visual mesh filename=package://a2_description/meshes/left_hind_Link4.stl
- link RL_hip: geometry visual mesh filename=package://a2_description/meshes/left_hind_Link1.stl
- link RL_thigh: geometry collision box size=0.017 0.05 0.05; collision box size=0.055 0.036 0.17
- link RR_calf: geometry collision box size=0.01 0.036 0.06; collision box size=0.02 0.036 0.06
- link RR_foot: geometry collision sphere radius=0.032; visual mesh filename=package://a2_description/meshes/right_hind_Link4.stl
- link RR_hip: geometry visual mesh filename=package://a2_description/meshes/right_hind_Link1.stl
- link RR_thigh: geometry collision box size=0.017 0.05 0.05; collision box size=0.055 0.036 0.17
- link base_link: geometry collision box size=0.045 0.1 0.01; collision box size=0.05 0.03 0.016
